Commit message: packages capable of chase-it final project

File: src/my_robot/urdf/my_robot.xacro (robot description, xacro)
@@ -1,5 +1,5 @@
 <?xml version='1.0'?>
 <robot name="my_robot" xmlns:xacro="http://www.ros.org/wiki/xacro">
-  <xacro:include filename="$(find my_bot)/urdf/my_bot.gazebo" />
+  <xacro:include filename="$(find my_robot)/urdf/my_robot.gazebo" />
   <link name="robot_footprint"></link>
   <joint name="robot_footprint_joint" type="fixed">
@@ -69,5 +69,5 @@
       />
     </inertial>
-    <visual name='left_visual'>
+    <visual name='left_wheel_visual'>
       <origin xyz="0.0 0 0.0" rpy=" 0 1.5707 1.5707"/>
       <geometry>
@@ -78,5 +78,5 @@
       </material>
     </visual>
-    <collision name='left_collision'>
+    <collision name='left_wheel_collision'>
         <origin xyz="0.0 0 0.0" rpy=" 0 1.5707 1.5707"/>
       <geometry>
@@ -107,5 +107,5 @@
       />
     </inertial>
-    <visual name='right_visual'>
+    <visual name='right_wheel_visual'>
       <origin xyz="0.0 0 0.0" rpy=" 0 1.5707 1.5707"/>
       <geometry>
@@ -116,5 +116,5 @@
       </material>
     </visual>
-    <collision name='right_collision'>
+    <collision name='right_wheel_collision'>
         <origin xyz="0.0 0 0.0" rpy=" 0 1.5707 1.5707"/>
       <geometry>
@@ -183,5 +183,5 @@
     <origin xyz="0.0 0 0.0" rpy=" 0 0 0"/>
       <geometry>
-        <mesh filename="package://my_bot/meshes/hokuyo.dae"/>
+        <mesh filename="package://my_robot/meshes/hokuyo.dae"/>
       </geometry>
     </visual>
@@ -201,13 +201,3 @@
   </joint>
   <!-- LIDAR joint -->
-    <!-- COLORING -->
-    <material name="orange">
-    <color rgba="${255/255} ${108/255} ${10/255} 1.0"/>
-    </material>
-    <gazebo reference="left_wheel">
-        <material>Gazebo/Orange</material>
-    </gazebo>
-    <gazebo reference="right_wheel">
-        <material>orange</material>
-    </gazebo>
 </robot>
